Commit message: 1

File: mujoco_simulation/model/robot_model/alexbot.urdf (robot description, URDF)
Before this commit: robot alexbot, 11 links, 10 joints
Links:
- link base_link: geometry collision mesh filename=/home/mr-cheng/Documents/Alexbot/mujoco_simulation/model/me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; visual mesh filename=/home/mr-cheng/Documents/Alexbot/mujoco_simulation/model/me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
- link leftlink1: geometry collision mesh filename=/home/mr-cheng/Documents/Alexbot/mujoco_simulation/model/me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; visual mesh filename=/home/mr-cheng/Documents/Alexbot/mujoco_simulation/model/me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
- link leftlink2: geometry collision mesh filename=/home/mr-cheng/Documents/Alexbot/mujoco_simulation/model/me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; visual mesh filename=/home/mr-cheng/Documents/Alexbot/mujoco_simulation/model/me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
- link leftlink3: geometry collision mesh filename=/home/mr-cheng/Documents/Alexbot/mujoco_simulation/model/me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; visual mesh filename=/home/mr-cheng/Documents/Alexbot/mujoco_simulation/model/me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
- link leftlink4: geometry collision mesh filename=/home/mr-cheng/Documents/Alexbot/mujoco_simulation/model/me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; visual mesh filename=/home/mr-cheng/Documents/Alexbot/mujoco_simulation/model/me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
- link leftlink5: geometry collision mesh filename=/home/mr-cheng/Documents/Alexbot/mujoco_simulation/model/me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; visual mesh filename=/home/mr-cheng/Documents/Alexbot/mujoco_simulation/model/me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
- link rightlink1: geometry collision mesh filename=/home/mr-cheng/Documents/Alexbot/mujoco_simulation/model/me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; visual mesh filename=/home/mr-cheng/Documents/Alexbot/mujoco_simulation/model/me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
- link rightlink2: geometry collision mesh filename=/home/mr-cheng/Documents/Alexbot/mujoco_simulation/model/me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; visual mesh filename=/home/mr-cheng/Documents/Alexbot/mujoco_simulation/model/me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
- link rightlink3: geometry collision mesh filename=/home/mr-cheng/Documents/Alexbot/mujoco_simulation/model/me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; visual mesh filename=/home/mr-cheng/Documents/Alexbot/mujoco_simulation/model/me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
- link rightlink4: geometry collision mesh filename=/home/mr-cheng/Documents/Alexbot/mujoco_simulation/model/me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; visual mesh filename=/home/mr-cheng/Documents/Alexbot/mujoco_simulation/model/me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
- link rightlink5: geometry collision mesh filename=/home/mr-cheng/Documents/Alexbot/mujoco_simulation/model/me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; visual mesh filename=/home/mr-cheng/Documents/Alexbot/mujoco_simulation/model/me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
